Commit message: Add theta-rho and change URDF to be more DH compatible.

File: urdf/theta_rho.urdf (robot description, URDF)
Before this commit: robot theta_rho, 9 links, 8 joints
Links:
- link tmp12: geometry collision cylinder length=0.0 radius=0.0; visual cylinder length=0.0 radius=0.0
Joints:
- joint a1: origin xyz=0.4 0 0 rpy=0 0 0 -> xyz=0.0 0 0 rpy=0 0 0
- joint a2: origin xyz=0.45 0 0 rpy=0 0 0 -> xyz=0.0 0 0 rpy=0 0 0
- joint alpha1: origin xyz=0 0 0 rpy=0 0 0 -> xyz=0 0 0 rpy=1.57 0 0
- joint alpha2: origin xyz=0 0 0 rpy=1.57 0 0 -> xyz=0 0 0 rpy=0.0 0 0
- joint d1: origin xyz=0 0 0 rpy=0 0 0 -> xyz=0 0 0.5 rpy=0 0 0
- joint d2: axis (none) -> 0 0 1; type fixed -> prismatic
- joint theta1: origin xyz=0 0 0 rpy=0 0 0 -> xyz=0 0 0 rpy=0 0 1.57
- joint theta2: axis 0 0 1 -> (none); limit lower=-3.1415 upper=3.1415 effort=1000.0 velocity=0.5 -> (none); origin xyz=0 0 0 rpy=0 0 0 -> xyz=0 0 0 rpy=0 0 1.57; type revolute -> fixed
